Commit message: robot_localization

File: robotx_description/urdf/robotx_base.urdf.xacro (robot description, xacro)
@@ -44,4 +44,26 @@
             </inertial>
         </link>
+    </xacro:macro>
+    <!-- support bars -->
+    <xacro:macro name="bars" params="position1 position2 sign_x sign_y sign_roll" >
+        <joint name="${position1}_${position2}_bar_joint" type="fixed">
+        <parent link="shelf_link"/>
+        <child link="${position1}_${position2}_bar_link"/>
+        <origin xyz="0 0 -${shelf_height/2}" rpy="0 0 0"/>
+    </joint>
+    <link name="${position1}_${position2}_bar_link">
+        <collision>
+            <origin xyz="${sign_x*shelf_length/2} ${sign_y*shelf_width/2} 0" rpy="${sign_roll*PI/8} 0 0"/>
+            <geometry>
+                <cylinder length="${shelf_height}" radius="0.01"/>
+            </geometry>
+        </collision>
+        <visual>
+            <origin xyz="${sign_x*shelf_length/2} ${sign_y*shelf_width/2} 0" rpy="${sign_roll*PI/8} 0 0"/>
+            <geometry>
+                <cylinder length="${shelf_height}" radius="0.01"/>
+            </geometry>
+        </visual>
+    </link>
     </xacro:macro>
     <!-- Base Link -->
@@ -100,4 +122,9 @@
         </inertial>
     </link>
+    <!-- bars -->
+    <xacro:bars position1="front" position2="left" sign_x="1" sign_y="-1" sign_roll="-1"/>
+    <xacro:bars position1="front" position2="right" sign_x="1" sign_y="1" sign_roll="1"/>
+    <xacro:bars position1="rear" position2="left" sign_x="-1" sign_y="-1" sign_roll="-1"/>
+    <xacro:bars position1="rear" position2="right" sign_x="-1" sign_y="1" sign_roll="1"/>
     <!-- sensor box joint-->
     <joint name="sensor_box_joint" type="fixed">

File: robotx_description/urdf/sensor.urdf.xacro (robot description, xacro)
@@ -74,6 +74,6 @@
     <xacro:spot_camera position1="front" position2="left" x="${shelf_length/2}" y="-${shelf_width/2}" yaw="0"/>
     <xacro:spot_camera position1="front" position2="right" x="${shelf_length/2}" y="${shelf_width/2}" yaw="0"/>
-    <xacro:spot_camera position1="middle" position2="left" x="0" y="-${shelf_width/2}" yaw="${PI/2}"/>
-    <xacro:spot_camera position1="middle" position2="right" x="0" y="${shelf_width/2}" yaw="-${PI/2}"/>
+    <xacro:spot_camera position1="middle" position2="left" x="0" y="-${shelf_width/2}" yaw="-${PI/2}"/>
+    <xacro:spot_camera position1="middle" position2="right" x="0" y="${shelf_width/2}" yaw="${PI/2}"/>
     <xacro:spot_camera position1="rear" position2="left" x="-${shelf_length/2}" y="-${shelf_width/2}" yaw="${PI}"/>
     <xacro:spot_camera position1="rear" position2="right" x="-${shelf_length/2}" y="${shelf_width/2}" yaw="${PI}"/>
