Commit message: vo for camera, unfinished tf

File: robotx_description/urdf/sensor.urdf.xacro (robot description, xacro)
@@ -10,8 +10,8 @@
         <joint name="${position1}_${position2}_camera_joint" type="fixed">
             <origin xyz="${x} ${y} ${shelf_thickness/2}" rpy="0 0 ${yaw}" />
-            <parent link="camera_array_link"/>
-            <child link="${position1}_${position2}_camera_link" />
+            <parent link="camera/array/link"/>
+            <child link="${position1}_stereo_${position2}_camera_link" />
         </joint>
-        <link name="${position1}_${position2}_camera_link">
+        <link name="${position1}_stereo_${position2}_camera_link">
             <visual>
                 <origin xyz="0 0 0" rpy="0 0 0" />
@@ -65,7 +65,7 @@
         <origin xyz="0 0 0" rpy="0 0 0" />
         <parent link="shelf_link"/>
-        <child link="camera_array_link"/>
+        <child link="camera/array/link"/>
     </joint>
-    <link name="camera_array_link" />
+    <link name="camera/array/link" />
     <xacro:imu position1="front" position2="left" x="${shelf_length/2}" y="-${shelf_width/2}" />
     <xacro:imu position1="front" position2="right" x="${shelf_length/2}" y="-${shelf_width/2}" />

Commit message: fix vo tf, still not finished

File: robotx_description/urdf/sensor.urdf.xacro (robot description, xacro)
@@ -10,8 +10,8 @@
         <joint name="${position1}_${position2}_camera_joint" type="fixed">
             <origin xyz="${x} ${y} ${shelf_thickness/2}" rpy="0 0 ${yaw}" />
-            <parent link="camera/array/link"/>
-            <child link="${position1}_stereo_${position2}_camera_link" />
+            <parent link="${position1}_stereo/camera_link"/>
+            <child link="${position1}_stereo/${position2}/camera_link" />
         </joint>
-        <link name="${position1}_stereo_${position2}_camera_link">
+        <link name="${position1}_stereo/${position2}/camera_link">
             <visual>
                 <origin xyz="0 0 0" rpy="0 0 0" />
@@ -62,10 +62,22 @@
     </joint>
     <link name="imu_array_link" />
-    <joint name="camera_array_joint" type="fixed">
+    <joint name="front_camera_array_joint" type="fixed">
         <origin xyz="0 0 0" rpy="0 0 0" />
         <parent link="shelf_link"/>
-        <child link="camera/array/link"/>
+        <child link="front_stereo/camera_link"/>
     </joint>
-    <link name="camera/array/link" />
+    <link name="front_stereo/camera_link" />
+    <joint name="mid_camera_array_joint" type="fixed">
+        <origin xyz="0 0 0" rpy="0 0 0" />
+        <parent link="shelf_link"/>
+        <child link="middle_stereo/camera_link"/>
+    </joint>
+    <link name="middle_stereo/camera_link" />
+    <joint name="rear_camera_array_joint" type="fixed">
+        <origin xyz="0 0 0" rpy="0 0 0" />
+        <parent link="shelf_link"/>
+        <child link="rear_stereo/camera_link"/>
+    </joint>
+    <link name="rear_stereo/camera_link" />
     <xacro:imu position1="front" position2="left" x="${shelf_length/2}" y="-${shelf_width/2}" />
     <xacro:imu position1="front" position2="right" x="${shelf_length/2}" y="-${shelf_width/2}" />

Commit message: modify camera and imu in gazebo

File: robotx_description/urdf/sensor.urdf.xacro (robot description, xacro)
@@ -6,8 +6,9 @@
     <xacro:property name="shelf_width" value="1.01" />
     <xacro:property name="shelf_thickness" value="0.1" />
+    <xacro:property name="camera_height" value="0.1" />
     <!-- Set up camera linkage and configuration -->
-    <xacro:macro name="spot_camera" params="position1 position2 x y yaw">
+    <xacro:macro name="spot_camera" params="position1 position2 x y z yaw">
         <joint name="${position1}_${position2}_camera_joint" type="fixed">
-            <origin xyz="${x} ${y} ${shelf_thickness/2}" rpy="0 0 ${yaw}" />
+            <origin xyz="${x} ${y} ${z+shelf_thickness/2}" rpy="0 0 ${yaw}" />
             <parent link="${position1}_stereo/camera_link"/>
             <child link="${position1}_stereo/${position2}/camera_link" />
@@ -80,14 +81,15 @@
     </joint>
     <link name="rear_stereo/camera_link" />
-    <xacro:imu position1="front" position2="left" x="${shelf_length/2}" y="-${shelf_width/2}" />
+    <xacro:imu position1="middle" position2="middle" x="0" y="0" />
+    <!--xacro:imu position1="front" position2="left" x="${shelf_length/2}" y="-${shelf_width/2}" />
     <xacro:imu position1="front" position2="right" x="${shelf_length/2}" y="-${shelf_width/2}" />
     <xacro:imu position1="rear" position2="left" x="${shelf_length/2}" y="-${shelf_width/2}" />
-    <xacro:imu position1="rear" position2="right" x="${shelf_length/2}" y="-${shelf_width/2}" />
-    <xacro:spot_camera position1="front" position2="left" x="${shelf_length/2}" y="-${shelf_width/2}" yaw="0"/>
-    <xacro:spot_camera position1="front" position2="right" x="${shelf_length/2}" y="${shelf_width/2}" yaw="0"/>
-    <xacro:spot_camera position1="middle" position2="left" x="0" y="-${shelf_width/2}" yaw="-${PI/2}"/>
-    <xacro:spot_camera position1="middle" position2="right" x="0" y="${shelf_width/2}" yaw="${PI/2}"/>
-    <xacro:spot_camera position1="rear" position2="left" x="-${shelf_length/2}" y="-${shelf_width/2}" yaw="${PI}"/>
-    <xacro:spot_camera position1="rear" position2="right" x="-${shelf_length/2}" y="${shelf_width/2}" yaw="${PI}"/>
+    <xacro:imu position1="rear" position2="right" x="${shelf_length/2}" y="-${shelf_width/2}" /-->
+    <xacro:spot_camera position1="front" position2="left" x="${shelf_length/2}" y="-${shelf_width/2}" z="${camera_height}" yaw="0"/>
+    <xacro:spot_camera position1="front" position2="right" x="${shelf_length/2}" y="${shelf_width/2}" z="${camera_height}" yaw="0"/>
+    <xacro:spot_camera position1="middle" position2="left" x="${shelf_length/2}" y="-${shelf_width/2}" z="0" yaw="-${PI/2}"/>
+    <xacro:spot_camera position1="middle" position2="right" x="${shelf_length/2}" y="${shelf_width/2}" z="0" yaw="${PI/2}"/>
+    <xacro:spot_camera position1="rear" position2="left" x="-${shelf_length/2}" y="-${shelf_width/2}" z="${camera_height}" yaw="-${PI/2}"/>
+    <xacro:spot_camera position1="rear" position2="right" x="-${shelf_length/2}" y="${shelf_width/2}" z="${camera_height}" yaw="${PI/2}"/>
     <!--kinect camera >
     <joint name="kinect_camera_joint" type="fixed">

Commit message: three pairs of stereo camera

File: robotx_description/urdf/sensor.urdf.xacro (robot description, xacro)
@@ -7,4 +7,13 @@
     <xacro:property name="shelf_thickness" value="0.1" />
     <xacro:property name="camera_height" value="0.1" />
+    <!-- camera array joint -->
+    <xacro:macro name="sport_camera_array" params="position1">
+        <joint name="${position1}_camera_array_joint" type="fixed">
+            <origin xyz="0 0 0" rpy="0 0 0" />
+            <parent link="shelf_link"/>
+            <child link="${position1}_stereo/camera_link"/>
+        </joint>
+        <link name="${position1}_stereo/camera_link"/>
+    </xacro:macro>
     <!-- Set up camera linkage and configuration -->
     <xacro:macro name="spot_camera" params="position1 position2 x y z yaw">
@@ -63,22 +72,4 @@
     </joint>
     <link name="imu_array_link" />
-    <joint name="front_camera_array_joint" type="fixed">
-        <origin xyz="0 0 0" rpy="0 0 0" />
-        <parent link="shelf_link"/>
-        <child link="front_stereo/camera_link"/>
-    </joint>
-    <link name="front_stereo/camera_link" />
-    <joint name="mid_camera_array_joint" type="fixed">
-        <origin xyz="0 0 0" rpy="0 0 0" />
-        <parent link="shelf_link"/>
-        <child link="middle_stereo/camera_link"/>
-    </joint>
-    <link name="middle_stereo/camera_link" />
-    <joint name="rear_camera_array_joint" type="fixed">
-        <origin xyz="0 0 0" rpy="0 0 0" />
-        <parent link="shelf_link"/>
-        <child link="rear_stereo/camera_link"/>
-    </joint>
-    <link name="rear_stereo/camera_link" />
     <xacro:imu position1="middle" position2="middle" x="0" y="0" />
     <!--xacro:imu position1="front" position2="left" x="${shelf_length/2}" y="-${shelf_width/2}" />
@@ -86,10 +77,13 @@
     <xacro:imu position1="rear" position2="left" x="${shelf_length/2}" y="-${shelf_width/2}" />
     <xacro:imu position1="rear" position2="right" x="${shelf_length/2}" y="-${shelf_width/2}" /-->
-    <xacro:spot_camera position1="front" position2="left" x="${shelf_length/2}" y="-${shelf_width/2}" z="${camera_height}" yaw="0"/>
-    <xacro:spot_camera position1="front" position2="right" x="${shelf_length/2}" y="${shelf_width/2}" z="${camera_height}" yaw="0"/>
-    <xacro:spot_camera position1="middle" position2="left" x="${shelf_length/2}" y="-${shelf_width/2}" z="0" yaw="-${PI/2}"/>
-    <xacro:spot_camera position1="middle" position2="right" x="${shelf_length/2}" y="${shelf_width/2}" z="0" yaw="${PI/2}"/>
-    <xacro:spot_camera position1="rear" position2="left" x="-${shelf_length/2}" y="-${shelf_width/2}" z="${camera_height}" yaw="-${PI/2}"/>
-    <xacro:spot_camera position1="rear" position2="right" x="-${shelf_length/2}" y="${shelf_width/2}" z="${camera_height}" yaw="${PI/2}"/>
+    <xacro:sport_camera_array position1="bow" />
+    <xacro:sport_camera_array position1="port" />
+    <xacro:sport_camera_array position1="starboard" />
+    <xacro:spot_camera position1="bow" position2="left" x="${shelf_length/2}" y="-${shelf_width/2}" z="${5*camera_height}" yaw="0"/>
+    <xacro:spot_camera position1="bow" position2="right" x="${shelf_length/2}" y="${shelf_width/2}" z="${5*camera_height}" yaw="0"/>
+    <xacro:spot_camera position1="port" position2="left" x="-${shelf_length/2}" y="-${shelf_width/2}" z="${camera_height}" yaw="-${PI/2}"/>
+    <xacro:spot_camera position1="port" position2="right" x="${shelf_length/2}" y="-${shelf_width/2}" z="${camera_height}" yaw="-${PI/2}"/>
+    <xacro:spot_camera position1="starboard" position2="left" x="${shelf_length/2}" y="${shelf_width/2}" z="${camera_height}" yaw="${PI/2}"/>
+    <xacro:spot_camera position1="starboard" position2="right" x="-${shelf_length/2}" y="${shelf_width/2}" z="${camera_height}" yaw="${PI/2}"/>
     <!--kinect camera >
     <joint name="kinect_camera_joint" type="fixed">
