Commit message: change gazebo test spawn and add triangle.xml

File: robotx_description/urdf/red_buoy.urdf (robot description, URDF)
Before this commit: robot green_buoy, 1 links, 0 joints
Links:
- removed link green_buoy
- added link red_buoy, mass 10.0; collision cylinder length=2 radius=0.5; visual mesh filename=package://robotx_description/meshes/green_buoy_marker.dae scale=1 1 1
