Commit message: dock

File: robotx_description/urdf/dock.urdf (robot description, URDF)
Before this commit: robot dock, 1 links, 0 joints
Links:
- removed link dock
- added link dock_base, mass 10.0; collision box size=14 1 0.01; visual mesh filename=package://robotx_description/meshes/dock_base.dae scale=1 1 1
- added link dock_wall, mass 10.0; collision box size=14 1 0.01; visual mesh filename=package://robotx_description/meshes/dock_wall.dae scale=1 1 1
- added link sign1, mass 1.0; collision box size=2 1 0.01; visual mesh filename=package://robotx_description/meshes/cross.dae scale=1 1 1
- added link sign2, mass 1.0; collision box size=2 1 0.01; visual mesh filename=package://robotx_description/meshes/circle.dae scale=1 1 1
- added link sign3, mass 1.0; collision box size=2 1 0.01; visual mesh filename=package://robotx_description/meshes/triangle.dae scale=1 1 1
Joints:
- added joint base_sign1_joint: type fixed, parent dock_base, child sign1, origin xyz=0 0 0
- added joint base_sign2_joint: type fixed, parent dock_base, child sign2, origin xyz=0 0 0
- added joint base_sign3_joint: type fixed, parent dock_base, child sign3, origin xyz=0 0 0
- added joint base_wall_joint: type fixed, parent dock_base, child dock_wall, origin xyz=0 0 0
