Commit message: gazebo for test2

File: robotx_description/urdf/blue_buoy.urdf (robot description, URDF)
Before this commit: robot red_buoy, 1 links, 0 joints
Links:
- removed link red_buoy
- added link blue_buoy, mass 10.0; collision cylinder length=2 radius=0.5; visual mesh filename=package://robotx_description/meshes/blue_buoy_marker.dae scale=1 1 1

File: robotx_description/urdf/dock.urdf (robot description, URDF)
Before this commit: robot red_buoy, 1 links, 0 joints
Links:
- removed link red_buoy
- added link dock, mass 1000.0; collision box size=10 5 0.01; visual mesh filename=package://robotx_description/meshes/dock.dae scale=1 1 1

File: robotx_description/urdf/yellow_buoy.urdf (robot description, URDF)
Before this commit: robot red_buoy, 1 links, 0 joints
Links:
- removed link red_buoy
- added link yellow_buoy, mass 10.0; collision cylinder length=2 radius=0.5; visual mesh filename=package://robotx_description/meshes/green_buoy_marker.dae scale=1 1 1

Commit message: change buoy collision dim

File: robotx_description/urdf/blue_buoy.urdf (robot description, URDF)
Before this commit: robot blue_buoy, 1 links, 0 joints
Links:
- link blue_buoy: geometry collision cylinder length=0.99 radius=0.127; visual mesh filename=package://robotx_description/meshes/blue_buoy_marker.dae scale=1 1 1

File: robotx_description/urdf/green_buoy.urdf (robot description, URDF)
Before this commit: robot green_buoy, 1 links, 0 joints
Links:
- link green_buoy: geometry collision cylinder length=0.99 radius=0.127; visual mesh filename=package://robotx_description/meshes/green_buoy_marker.dae scale=1 1 1

File: robotx_description/urdf/red_buoy.urdf (robot description, URDF)
Before this commit: robot red_buoy, 1 links, 0 joints
Links:
- link red_buoy: geometry collision cylinder length=0.99 radius=0.127; visual mesh filename=package://robotx_description/meshes/red_buoy_marker.dae scale=1 1 1

File: robotx_description/urdf/yellow_buoy.urdf (robot description, URDF)
Before this commit: robot yellow_buoy, 1 links, 0 joints
Links:
- link yellow_buoy: geometry collision cylinder length=0.99 radius=0.127; visual mesh filename=package://robotx_description/meshes/green_buoy_marker.dae scale=1 1 1

Commit message: move base and gazebo

File: robotx_description/urdf/blue_buoy.urdf (robot description, URDF)
Before this commit: robot blue_buoy, 1 links, 0 joints
Links:
- link blue_buoy: geometry collision cylinder length=0.99 radius=0.127; visual mesh filename=package://robotx_description/meshes/totem_cap.dae scale=1 1 1

File: robotx_description/urdf/green_buoy.urdf (robot description, URDF)
Before this commit: robot green_buoy, 1 links, 0 joints
Links:
- link green_buoy: geometry collision cylinder length=0.99 radius=0.127; visual mesh filename=package://robotx_description/meshes/totem_flat.dae scale=1 1 1

File: robotx_description/urdf/red_buoy.urdf (robot description, URDF)
Before this commit: robot red_buoy, 1 links, 0 joints
Links:
- link red_buoy: geometry collision cylinder length=0.99 radius=0.127; visual mesh filename=package://robotx_description/meshes/totem_cap.dae scale=1 1 1

File: robotx_description/urdf/yellow_buoy.urdf (robot description, URDF)
Before this commit: robot yellow_buoy, 1 links, 0 joints
Links:
- link yellow_buoy: geometry collision cylinder length=0.99 radius=0.127; visual mesh filename=package://robotx_description/meshes/totem_flat.dae scale=1 1 1
